File: PCB/HB-ES-PMSw1-USB.kicad_pcb (KiCad board)
At the start: 2 copper layers, 70.2 x 27.7 mm, 42 parts, among them J1 FTDI, J2 USB_B_Micro, J3 USB_A, J4 ISP, Q1 BC847C, SW1 Config, U1 CC1101, U2 INA219, U3 MCP1700-3302, U4 ATmega328P-AU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

Commit message: update kicad
Other:
- net class 1 removed
- net class Default removed
